Commit message: GripperIssue: added custom franka description Camera: added simulated depth camera

File: src/custom_franka_description/end_effectors/common/ee_with_one_link.xacro (robot description, xacro)
@@ -2,5 +2,5 @@
 <robot xmlns:xacro="http://www.ros.org/wiki/xacro" name="ee_with_one_link">
   <!-- safety_distance: Minimum safety distance in [m] by which the collision volumes are expanded and which is enforced during robot motions -->
-  <xacro:macro name="ee_with_one_link" params="connected_to:='' robot_type arm_prefix:='' ee_id ee_inertials rpy_ee:='0 0 0' xyz_ee:='0 0 0' tcp_xyz:='0 0 0' tcp_rpy:='0 0 0' safety_distance:=0 gazebo:=false description_pkg:=franka_description with_sc:=false">
+  <xacro:macro name="ee_with_one_link" params="connected_to:='' robot_type arm_prefix:='' ee_id ee_inertials rpy_ee:='0 0 0' xyz_ee:='0 0 0' tcp_xyz:='0 0 0' tcp_rpy:='0 0 0' safety_distance:=0 gazebo:=false description_pkg:=custom_franka_description with_sc:=false">
     <xacro:property name="ee_prefix" default="robot_"/>
     <xacro:unless value="${robot_type == ''}">

File: src/custom_franka_description/end_effectors/common/franka_hand.xacro (robot description, xacro)
@@ -12,5 +12,5 @@
                        safety_distance:=0
                        gazebo:=false
-                       description_pkg:=franka_description
+                       description_pkg:=custom_franka_description
                        with_sc:=false
                        no_prefix:=false">

File: src/custom_franka_description/end_effectors/common/utils.xacro (robot description, xacro)
@@ -42,5 +42,5 @@
       <collision name="${prefix}${name}_collision">
         <geometry>
-          <mesh filename="package://franka_description/meshes/robot_ee/${ee_id}/collision/${name}.stl" />
+          <mesh filename="package://custom_franka_description/meshes/robot_ee/${ee_id}/collision/${name}.stl" />
         </geometry>
       </collision>

File: src/custom_franka_description/end_effectors/franka_hand/franka_hand.urdf.xacro (robot description, xacro)
@@ -1,11 +1,11 @@
 <?xml version="1.0" encoding="utf-8"?>
 <robot xmlns:xacro="http://www.ros.org/wiki/xacro" name="franka_hand">
-  <xacro:include filename="$(find franka_description)/end_effectors/common/utils.xacro" />
-  <xacro:include filename="$(find franka_description)/end_effectors/common/franka_hand.xacro"/>
-  <xacro:include filename="$(find franka_description)/end_effectors/franka_hand/franka_hand_arguments.xacro"/>
+  <xacro:include filename="$(find custom_franka_description)/end_effectors/common/utils.xacro" />
+  <xacro:include filename="$(find custom_franka_description)/end_effectors/common/franka_hand.xacro"/>
+  <xacro:include filename="$(find custom_franka_description)/end_effectors/franka_hand/franka_hand_arguments.xacro"/>
   <xacro:franka_hand connected_to="$(arg special_connection)"
                      robot_type="$(arg robot_type)"
                      ee_id="$(arg ee_id)_$(arg ee_color)"
-                     ee_inertials="${xacro.load_yaml('$(find franka_description)/end_effectors/$(arg ee_id)/inertials.yaml')}"
+                     ee_inertials="${xacro.load_yaml('$(find custom_franka_description)/end_effectors/$(arg ee_id)/inertials.yaml')}"
                      rpy_ee="$(arg rpy_ee)"
                      xyz_ee="$(arg xyz_ee)"

File: src/custom_franka_description/end_effectors/franka_hand/franka_hand_arguments.xacro (robot description, xacro)
@@ -24,4 +24,4 @@
   <xacro:arg name="gazebo" default="false" />
   <!-- Name of the description package -->
-  <xacro:arg name="description_pkg" default="franka_description" />
+  <xacro:arg name="description_pkg" default="custom_franka_description" />
 </robot>

File: src/custom_franka_description/robots/common/franka_arm.xacro (robot description, xacro)
@@ -1,17 +1,17 @@
 <?xml version='1.0' encoding='utf-8'?>
 <robot xmlns:xacro="http://www.ros.org/wiki/xacro" name="franka_arm">
-  <xacro:include filename="$(find franka_description)/robots/common/utils.xacro" />
+  <xacro:include filename="$(find custom_franka_description)/robots/common/utils.xacro" />
   <!-- safety_distance: Minimum safety distance in [m] by which the collision volumes are expanded and which is enforced during robot motions -->
   <!-- robot_type: the franka robot arm type -->
-  <!-- joint_limits: description of the joint limits that comes from a YAML file. Example definition: ${xacro.load_yaml('$(find franka_description)/robots/fr3/joint_limits.yaml')} -->
-  <!-- kinematics: description of the kinematics that comes from a YAML file. Example definition: ${xacro.load_yaml('$(find franka_description)/robots/fr3/kinematics.yaml')} -->
-  <!-- inertials: description of the inertials that comes from a YAML file. Example definition: ${xacro.load_yaml('$(find franka_description)/robots/fr3/inertials.yaml')} -->
-  <!-- dynamics: description of the dynamics that comes from a YAML file. Example definition: ${xacro.load_yaml('$(find franka_description)/robots/fr3/dynamics.yaml')} -->
-  <xacro:macro name="franka_arm" params="robot_type arm_prefix:='' no_prefix:=false description_pkg:='franka_description' connected_to:='base' xyz:='0 0 0' rpy:='0 0 0' gazebo:='false' safety_distance:=0 with_sc:=false" >
-    <xacro:property name="joint_limits" value="${xacro.load_yaml('$(find franka_description)/robots/' + robot_type + '/joint_limits.yaml')}"/>
-    <xacro:property name="inertials" value="${xacro.load_yaml('$(find franka_description)/robots/' + robot_type  + '/inertials.yaml')}"/>
-    <xacro:property name="kinematics" value="${xacro.load_yaml('$(find franka_description)/robots/' + robot_type + '/kinematics.yaml')}"/>
-    <xacro:property name="accelerometer_config" value="${xacro.load_yaml('$(find franka_description)/robots/' + robot_type + '/accelerometers.yaml')}"/>
-    <xacro:property name="dynamics" value="${xacro.load_yaml('$(find franka_description)/robots/' + robot_type + '/dynamics.yaml')}"/>
+  <!-- joint_limits: description of the joint limits that comes from a YAML file. Example definition: ${xacro.load_yaml('$(find custom_franka_description)/robots/fr3/joint_limits.yaml')} -->
+  <!-- kinematics: description of the kinematics that comes from a YAML file. Example definition: ${xacro.load_yaml('$(find custom_franka_description)/robots/fr3/kinematics.yaml')} -->
+  <!-- inertials: description of the inertials that comes from a YAML file. Example definition: ${xacro.load_yaml('$(find custom_franka_description)/robots/fr3/inertials.yaml')} -->
+  <!-- dynamics: description of the dynamics that comes from a YAML file. Example definition: ${xacro.load_yaml('$(find custom_franka_description)/robots/fr3/dynamics.yaml')} -->
+  <xacro:macro name="franka_arm" params="robot_type arm_prefix:='' no_prefix:=false description_pkg:='custom_franka_description' connected_to:='base' xyz:='0 0 0' rpy:='0 0 0' gazebo:='false' safety_distance:=0 with_sc:=false" >
+    <xacro:property name="joint_limits" value="${xacro.load_yaml('$(find custom_franka_description)/robots/' + robot_type + '/joint_limits.yaml')}"/>
+    <xacro:property name="inertials" value="${xacro.load_yaml('$(find custom_franka_description)/robots/' + robot_type  + '/inertials.yaml')}"/>
+    <xacro:property name="kinematics" value="${xacro.load_yaml('$(find custom_franka_description)/robots/' + robot_type + '/kinematics.yaml')}"/>
+    <xacro:property name="accelerometer_config" value="${xacro.load_yaml('$(find custom_franka_description)/robots/' + robot_type + '/accelerometers.yaml')}"/>
+    <xacro:property name="dynamics" value="${xacro.load_yaml('$(find custom_franka_description)/robots/' + robot_type + '/dynamics.yaml')}"/>
     <!-- Define a property that defaults to 'arm_prefix_robot_type' concatenated with an underscore if 'no_prefix' is not set -->
     <xacro:property name="prefix" value="${'' if no_prefix else arm_prefix + robot_type + '_'}" />

File: src/custom_franka_description/robots/common/utils.xacro (robot description, xacro)
@@ -43,5 +43,5 @@
       <collision name="${prefix}${name}_collision">
         <geometry>
-          <mesh filename="package://franka_description/meshes/robots/${robot_type}/collision/${name}.stl" />
+          <mesh filename="package://custom_franka_description/meshes/robots/${robot_type}/collision/${name}.stl" />
         </geometry>
       </collision>

File: src/custom_franka_description/robots/fr3/fr3.srdf.xacro (robot description, xacro)
@@ -1,5 +1,5 @@
 <?xml version='1.0' encoding='utf-8'?>
 <robot xmlns:xacro="http://www.ros.org/wiki/xacro" name="fr3">
-  <xacro:include filename="$(find franka_description)/robots/common/franka_arm.srdf.xacro"/>
+  <xacro:include filename="$(find custom_franka_description)/robots/common/franka_arm.srdf.xacro"/>
   <!-- The ID of the robot model to be used -->
   <xacro:arg name="robot_type" default="fr3" />

File: src/custom_franka_description/robots/fr3/fr3.urdf.xacro (robot description, xacro)
@@ -1,5 +1,5 @@
 <?xml version="1.0" encoding="utf-8"?>
 <robot xmlns:xacro="http://www.ros.org/wiki/xacro" name="fr3">
-  <xacro:include filename="$(find franka_description)/robots/common/franka_robot.xacro"/>
+  <xacro:include filename="$(find custom_franka_description)/robots/common/franka_robot.xacro"/>
   <!-- Define arguments -->
   <!-- The ID of the robot model to be used -->
@@ -40,5 +40,5 @@
   <xacro:arg name="gazebo_effort" default="false"/>
   <!-- Name of the description package -->
-  <xacro:arg name="description_pkg" default="franka_description"/>
+  <xacro:arg name="description_pkg" default="custom_franka_description"/>
   <!-- Append an underscore to the user-provided prefix, if non-empty. -->
   <xacro:property name="prefix" value="$(arg arm_prefix)"/>
